File: Solar_NYHL/Solar_NYHL.sch (KiCad schematic (older format))
At the start: 12 parts

Commit message: 0. Draft
kezdetleges lábkiosztás
Parts:
- removed XA?: Arduino_Mega2560_Shield, Arduino:Arduino_Mega2560_Shield, symbol Solar_NYHL-rescue:Arduino_Mega2560_Shield-arduino
- added H1, H2, H3, H4, H5, H6: MountingHole, symbol Mechanical:MountingHole
- gave numbers to parts that had none: 11
Connections:
- net 3V3a is gone; now on an unnamed net: J3.4 (Pin_4)
- net 5Vb is gone; now on an unnamed net: J4.36 (Pin_36)
- net 5Vc is gone; now on an unnamed net: J4.1 (Pin_1)
- net D18 is gone; now on an unnamed net: J6.4 (Pin_4)
- net D19 is gone; now on an unnamed net: J6.3 (Pin_3)
- net D20 is gone; now on an unnamed net: J6.2 (Pin_2)
- net D21 is gone; now on an unnamed net: J6.1 (Pin_1)
- net D23 is gone; now on an unnamed net: J4.35 (Pin_35)
- net D51 is gone; now on an unnamed net: J4.21 (Pin_21)
- net D53 is gone; now on an unnamed net: J4.20 (Pin_20)
- net GNDc is gone; now on an unnamed net: J4.18 (Pin_18)
- net GNDd is gone; now on an unnamed net: J4.19 (Pin_19)
- net GNDe is gone; now on an unnamed net: J7.7 (Pin_7)
- net at U2.2 (SCK): now also J4.17 (Pin_17)
- net at U2.4 (SO): now also J4.16 (Pin_16)
- removed net D52: J4.16 (Pin_16), J4.17 (Pin_17)
- no-connect marks 1 -> 11
Other:
- note added: "3V3a"
- note added: "5V"
- note added: "5Vb"
- note added: "Analog1"
- note added: "Analog2"
- note added: "D18"
- note added: "D19"
- note added: "D20"
- note added: "D21"
- note added: "D23"
- note added: "GNDc"
- note added: "GNDd"
- note added: "GNDe"
- note added: "Mounting holes"
- note added: "PWM"
- note added: "RXD1, INT2 (D19)"
- note added: "TXD1, INT3 (D18)"
- note added: "UART1_RxD"
- note added: "UART2_TxD"
- note added: "arduino MISO"
- note added: "arduino MISO\n"
- note added: "arduino MOSI"
- note added: "arduino SCK"
- note added: "arduino SCL (D21)"
- note added: "arduino SDA (D20)"
- note added: "arduino SS"
- moved on the sheet: J2, J7, U1, U2, U3
